File: MPO21.brd (EAGLE design)
At the start: 92.1 x 58.7 mm, 42 parts, among them J1 JTAG, J4 CONN_20X2NOSILK, J9 USB Female Type C Connector, Q1 DMP1045U, U1 ATSAMD21G-A, U3 3.3V, U4 MCP73831, U5 XTSD, X1 SM03B-SRSS-TB, Y1 32.768kHz

Commit message: propeller yo
Parts:
- removed C17, C18: 0.1uF, rcl:C0603
- removed C19: 1uF, rcl:C0603
- removed C20, C21: 22pF, rcl:C0603
- removed I2C1: QWIIC_RIGHT_ANGLE, SparkFun-Connectors:JST04_1MM_RA
- removed J1: JTAG, SparkFun-Connectors:2X5-SMD-1.27MM
- removed J8: (no value), SparkFun-Connectors:1X05_LOCK
- removed X1: SM03B-SRSS-TB, con-JST:SM03B-SRSS-TB
- removed Y1: 32.768kHz, SparkFun-Clocks:CRYSTAL-SMD-2X6-CYL
- added IC1, IC2, IC3, IC4: (no value), linear:SO14
- added QG1: SM77H, crystal:SM77H
- added U$2: PROPELLER-44Q, Parallax:Q44
- added U2, U6: W25Q32FV, SparkFun-IC-Memory:SOIC-8
- U1: value ATSAMD21G-A -> W25Q32FV; device SparkFun-IC-Microcontroller:TQFP-48 -> SparkFun-IC-Memory:SOIC-8
- U5: value XTSD -> W25Q32FV; device microbuilder:LGA8_8X6 -> SparkFun-IC-Memory:SOIC-8
- moved R20 32.9 mm to (31.8, 70.2)
- moved R21 32.9 mm to (31.8, 68.6)
- moved I2C2 21.6 mm to (14.0, 72.7)
- moved U1 12.8 mm to (62.2, 62.2), turned to 270 degrees
- moved U5 9.21 mm to (62.2, 55.9), turned to 270 degrees
Connections:
- removed net N$1: U5.3
- removed net N$14: U1.17
- removed net N$15: U1.44
- removed net N$2: U5.5
- removed net N$42: U5.7
- removed net N$64: J1.7
- removed net N$7: U5.6
- removed net N$70: J1.8
- removed net N$8: U5.2
- removed net N$9: U5.1
- removed net PA00: C20.2, U1.1, Y1.X2
- removed net PA02: U1.3
- removed net PA03: U1.4
- removed net PA04: U1.9
- removed net PA05: U1.10
- removed net PA06: U1.11
- removed net PA07: U1.12
- removed net PA10: U1.15
- removed net PA11: U1.16
- removed net PA12: U1.21
- removed net PA13: U1.22
- removed net PA14: U1.23
- removed net PA15: U1.24
- removed net PA16: U1.25
- removed net PA17: U1.26
- removed net PA18: U1.27
- removed net PA19: U1.28
- removed net PA20: U1.29
- removed net PA21: U1.30
- removed net PA22: I2C1.3, U1.31
- removed net PA23: I2C1.4, U1.32
- removed net PA27: U1.39
- removed net PA28: U1.41
- removed net PB02: U1.47
- removed net PB03: U1.48
- removed net PB08: U1.7
- removed net PB09: U1.8
- removed net PB10: U1.19
- removed net PB11: U1.20
- removed net PB22: U1.37
- removed net PB23: U1.38
- removed net RST: J1.10, U1.40
- removed net SWCLK: J1.4, U1.45, X1.1
- removed net SWDIO: J1.2, U1.46, X1.3
- removed net SWO: J1.6
- removed net VDDCORE: C18.1, U1.43
- new net AGND: IC1.8, IC2.8, IC3.8, IC4.8
- new net DGND: IC1.7, IC2.7, IC3.7, IC4.7
- new net VCC: IC1.14, IC2.14, IC3.14, IC4.14, QG1.4
- new net VDD: U$2.18, U$2.30, U$2.40, U$2.8
- new net VSS: U$2.17, U$2.27, U$2.39, U$2.5
- net D+: no longer U1.34
- net D-: no longer U1.33
- net GND: now also QG1.2; no longer C17.1, C18.2, C19.1, C20.1, C21.1, I2C1.1, J1.3, J1.5, J1.9, U1.18, U1.35, U1.42, U1.5, U5.4, X1.2
- net PA01: no longer C21.2, U1.2, Y1.X1
- net PA08: no longer U1.13
- net PA09: no longer U1.14
- net VIN_UC: no longer C17.2, C19.2, I2C1.2, J1.1, U1.36, U1.6, U5.8
