File: MPO21.sch (EAGLE design)
At the start: 42 parts, among them J1 JTAG, J4 CONN_20X2NOSILK, J9 USB Female Type C Connector, Q1 DMP1045U, U1 ATSAMD21G-A, U3 3.3V, U4 MCP73831, U5 XTSD, X1 SM03B-SRSS-TB, Y1 32.768kHz

Commit message: propeller yo
Parts:
- removed C17, C18: 0.1uF, rcl:C-EUC0603
- removed C19: 1uF, rcl:C-EUC0603
- removed C20, C21: 22pF, rcl:C-EUC0603
- removed I2C1: QWIIC_RIGHT_ANGLE, SparkFun-Connectors:QWIIC_CONNECTORJS-1MM
- removed J1: JTAG, SparkFun-Connectors:CORTEX_JTAG_DEBUG_SMD
- removed J8: (no value), SparkFun-Connectors:CONN_05LOCK
- removed X1: SM03B-SRSS-TB, con-JST:SM03B-SRSS-TB
- removed Y1: 32.768kHz, SparkFun-Clocks:CRYSTAL-32.768KHZSMD-2X6
- added IC1, IC2, IC3, IC4: (no value), linear:ADC08034D
- added QG1: SM77H, crystal:SM77H
- added U$2: PROPELLER-44Q, Parallax:PROPELLER-44Q
- added U2, U6: W25Q32FV, SparkFun-IC-Memory:W25Q32FVSS
- U1: value ATSAMD21G-A -> W25Q32FV; device SparkFun-IC-Microcontroller:ATSAMD21G-A -> SparkFun-IC-Memory:W25Q32FVSS
- U5: value XTSD -> W25Q32FV; device microbuilder:SMT_SDCARD_8PIN -> SparkFun-IC-Memory:W25Q32FVSS
Connections:
- removed net N$1: U5.SCK
- removed net N$14: U1.VDDIO@17
- removed net N$15: U1.VDDIN
- removed net N$2: U5.MOSI/CMD
- removed net N$42: U5.SD1
- removed net N$64: J1.KEY
- removed net N$7: U5.MISO/SD0
- removed net N$70: J1.NC/TDI
- removed net N$8: U5.SSEL/SD3
- removed net N$9: U5.SD2
- removed net PA00: C20.2, U1.PA00(XIN32/SER1:0/TC2:0), Y1.2
- removed net PA02: U1.A0_PA02(AIN0/DAC)
- removed net PA03: U1.PA03(AIN1/REFA)
- removed net PA04: U1.A3_PA04(AIN4/REFB/SER0:0/TC0:0)
- removed net PA05: U1.A4_PA05(AIN5/SER0:1/TC0:1)
- removed net PA06: U1.D8_PA06(AIN6/SER0:2/TC1:0)
- removed net PA07: U1.D9_PA07(AIN7/SER0:3/TC1:1)
- removed net PA10: U1.PA10(AIN18/SER0:2+)_D1/TX
- removed net PA11: U1.PA11(AIN19/SER0:3+)_D0/RX
- removed net PA12: U1.PA12(I2C/SER2:0+)_MISO
- removed net PA13: U1.PA13(I2C/SER2:1+)
- removed net PA14: U1.PA14(XIN/SER2:2+)_D2
- removed net PA15: U1.PA15(XOUT/SER2:3+)_D5
- removed net PA16: U1.PA16(I2C/SER1:0+)_D11
- removed net PA17: U1.PA17(I2C/SER1:1+)_D13
- removed net PA18: U1.PA18(SER1:2+)_D10
- removed net PA19: U1.PA19(SER1:3+)_D12
- removed net PA20: U1.PA20(SER5:2+)_D6
- removed net PA21: U1.PA21(SER5:3+)_D7
- removed net PA22: I2C1.3, U1.PA22(I2C/SER3:0+)_SDA
- removed net PA23: I2C1.4, U1.PA23(I2C/SER3:0+)_SCL
- removed net PA27: U1.PA27
- removed net PA28: U1.PA28
- removed net PB02: U1.A5_PB02(AIN10/SER5:0)
- removed net PB03: U1.PB03(AIN11/SER5:1)
- removed net PB08: U1.A1_PB08(AIN2/SER4:0/TC4:0)
- removed net PB09: U1.A2_PB09(AIN3/SER4:1/TC4:1)
- removed net PB10: U1.PB10(SER4:2+)_MOSI
- removed net PB11: U1.PB11(SER4:3+)_SCK
- removed net PB22: U1.PB22(SER5:2+)
- removed net PB23: U1.PB23(SER5:3+)
- removed net RST: J1.!RESET, U1.!RESET!
- removed net SWCLK: J1.SWDCLK/TCK, U1.PA30(SWCLK/SER1:2+), X1.1
- removed net SWDIO: J1.SWDIO/TMS, U1.PA31(SWDIO/SER1:3+), X1.3
- removed net SWO: J1.SWO/TDO
- removed net VDDCORE: C18.1, U1.VDDCORE
- net D+: no longer U1.PA25(SER3:3+)
- net D-: no longer U1.PA24(SER3:2+)
- net GND: no longer C17.1, C18.2, C19.1, C20.1, C21.1, I2C1.1, J1.GND@3, J1.GND@5, J1.GNDDTCT, U1.GND@18, U1.GND@35, U1.GND@42, U1.GNDANA, U5.VSS, X1.2
- net PA01: no longer C21.2, U1.PA01(XOUT32/SER1:1/TC2:1), Y1.1
- net PA08: no longer U1.PA08(I2C/AIN16/SER0:0+)_D4
- net PA09: no longer U1.PA09(I2C/AIN17/SER0:1+)_D3
- net VIN_UC: no longer C17.2, C19.2, I2C1.2, J1.VCC, U1.VDDANA, U1.VDDIO@36, U5.VCC
Other:
- moved on the sheet: U5
